File: hardware/snes-to-db9-controller-adapter/adapter.sch (EAGLE design)
At the start: 5 parts, among them IC1 MEGA8-P

Commit message: Update SNES to DB9 adapter
Parts:
- added JP1: (no value), jumper:JP1E
Connections:
- new net N$1: IC1.PD6(AIN0), JP1.2
- net GND: now also JP1.1
Changed lines of the file:
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@@
 <part name="P+3" library="supply1" library_urn="urn:adsk.eagle:library:371" deviceset="VCC" device=""/>
 <part name="GND4" library="supply1" library_urn="urn:adsk.eagle:library:371" deviceset="GND" device=""/>
+<part name="JP1" library="jumper" library_urn="urn:adsk.eagle:library:252" deviceset="JP1E" device="" package3d_urn="urn:adsk.eagle:package:15455/1"/>
 </parts>
 <sheets>
@@
 <instance part="GND4" gate="1" x="104.14" y="33.02" smashed="yes" rot="R180">
 <attribute name="VALUE" x="106.68" y="35.56" size="1.778" layer="96" rot="R180"/>
+</instance>
+<instance part="JP1" gate="A" x="96.52" y="30.48" smashed="yes" rot="R180">
+<attribute name="NAME" x="97.79" y="30.48" size="1.778" layer="95" rot="R270"/>
+<attribute name="VALUE" x="90.805" y="30.48" size="1.778" layer="96" rot="R270"/>
 </instance>
 </instances>
@@
 <pinref part="GND4" gate="1" pin="GND"/>
 <wire x1="104.14" y1="22.86" x2="104.14" y2="30.48" width="0.1524" layer="91"/>
+<wire x1="104.14" y1="30.48" x2="99.06" y2="30.48" width="0.1524" layer="91"/>
+<junction x="104.14" y="30.48"/>
+<wire x1="99.06" y1="30.48" x2="99.06" y2="33.02" width="0.1524" layer="91"/>
+<pinref part="JP1" gate="A" pin="1"/>
+<wire x1="99.06" y1="33.02" x2="96.52" y2="33.02" width="0.1524" layer="91"/>
 </segment>
 </net>
@@
 </segment>
 </net>
+<net name="N$1" class="0">
+<segment>
+<pinref part="JP1" gate="A" pin="2"/>
+<wire x1="93.98" y1="33.02" x2="93.98" y2="38.1" width="0.1524" layer="91"/>
+<pinref part="IC1" gate="G$1" pin="PD6(AIN0)"/>
+<wire x1="93.98" y1="38.1" x2="76.2" y2="38.1" width="0.1524" layer="91"/>
+</segment>
+</net>
