File: hardware/snes-to-db9-controller-adapter/adapter.brd (EAGLE design)
At the start: 38 x 40 mm, 5 parts, among them IC1 MEGA8-P

Commit message: Update SNES to DB9 adapter
Parts:
- added JP1: (no value), jumper:JP1
Connections:
- new net N$1: IC1.12, JP1.2
- net GND: now also JP1.1
Routing:
- net GND: track 45.9 -> 51.8 mm
- net N$1: track 0.00 -> 4.49 mm
- added copper zone on layer 1, net GND
- added copper zone on layer 16, net GND
Changed lines of the file:
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@@
 <attribute name="VALUE" x="20.32" y="32.4" size="1.778" layer="27" ratio="10"/>
+</element>
+<element name="JP1" library="jumper" library_urn="urn:adsk.eagle:library:252" package="JP1" package3d_urn="urn:adsk.eagle:package:15455/1" value="" x="34" y="8" smashed="yes" rot="R90">
+<attribute name="NAME" x="36.54" y="6.349" size="1.27" layer="25" ratio="10" rot="R180"/>
+<attribute name="POPULARITY" value="61" x="34" y="8" size="1.778" layer="27" rot="R90" display="off"/>
+<attribute name="VALUE" x="36.54" y="10.921" size="1.27" layer="27" ratio="10" rot="R180"/>
 </element>
 </elements>
@@
 <wire x1="19" y1="18" x2="19" y2="35.5" width="0.1524" layer="16"/>
 <wire x1="20" y1="36.5" x2="20.4216" y2="36.5148" width="0.1524" layer="16"/>
-<wire x1="27.5" y1="7.5" x2="32" y2="3" width="0.1524" layer="1"/>
+<wire x1="27.5" y1="7.5" x2="31" y2="4" width="0.1524" layer="1"/>
+<wire x1="31" y1="4" x2="32" y2="3" width="0.1524" layer="1"/>
 <wire x1="21" y1="7.5" x2="27.5" y2="7.5" width="0.1524" layer="1"/>
 <wire x1="32" y1="3" x2="32.28" y2="2.54" width="0.1524" layer="1"/>
 <wire x1="21" y1="7.5" x2="20.87" y2="7.88" width="0.1524" layer="1"/>
+<contactref element="JP1" pad="1"/>
+<wire x1="31" y1="4" x2="35" y2="8" width="0.1524" layer="1"/>
+<wire x1="35" y1="8" x2="35.27" y2="8" width="0.1524" layer="1"/>
+<polygon width="0.1524" layer="1">
+<vertex x="-1" y="41"/>
+<vertex x="38" y="41"/>
+<vertex x="39" y="40"/>
+<vertex x="39" y="-1"/>
+<vertex x="-1" y="-1"/>
+</polygon>
+<polygon width="0.1524" layer="16">
+<vertex x="-3" y="42"/>
+<vertex x="39" y="42"/>
+<vertex x="40" y="41"/>
+<vertex x="40" y="-1"/>
+<vertex x="-3" y="-1"/>
+</polygon>
 </signal>
 <signal name="N$2">
@@
 <wire x1="23" y1="36.5" x2="23.1648" y2="36.5148" width="0.1524" layer="16"/>
 </signal>
+<signal name="N$1">
+<contactref element="JP1" pad="2"/>
+<contactref element="IC1" pad="12"/>
+<wire x1="32.5" y1="9" x2="30.5" y2="11" width="0.1524" layer="1"/>
+<wire x1="32.5" y1="8" x2="32.5" y2="9" width="0.1524" layer="1"/>
+<wire x1="30.5" y1="11" x2="30.48" y2="11.43" width="0.1524" layer="1"/>
+<wire x1="32.5" y1="8" x2="32.73" y2="8" width="0.1524" layer="1"/>
+</signal>
 </signals>

Commit message: Update SNES to DB9 adapter
Parts:
- moved R1 25.4 mm to (30.3, 19.9), turned to 0 degrees
- moved JP1 13.6 mm to (21.0, 4.00), turned to 180 degrees
- moved C1 12.2 mm to (19.4, 20.1), turned to 0 degrees
- moved IC1 2.48 mm to (18.9, 12.8), turned to 180 degrees
Routing:
- net FIRE: track 61.9 -> 32.4 mm
- net SECOND_FIRE: track 18.6 -> 40.9 mm, vias 1 -> 0
- net UP: track 43.2 -> 25.9 mm
- net N$1: track 4.49 -> 20.4 mm
- net VCC: track 61.5 -> 75.5 mm
- net RIGHT: track 21.2 -> 33.5 mm
- net DATA: track 23.3 -> 12.9 mm
- net LEFT: track 28.9 -> 33.4 mm
- net LATCH: track 17.2 -> 14.3 mm, vias 1 -> 0
- net GND: track 51.8 -> 49.1 mm, vias 0 -> 1
- net THIRD_FIRE: track 27.5 -> 28.8 mm
- net CLK: track 21.3 -> 20.2 mm, vias 1 -> 0
- net DOWN: track 34.3 -> 33.4 mm
Other:
- board size 38 x 40 mm -> 38 x 39 mm

Commit message: Update SNES to DB9 adapter
Parts:
- moved JP1 19.9 mm to (19.0, 23.8), turned to 270 degrees
- moved C1 0.57 mm to (19.0, 19.7)
Routing:
- net VCC: track 75.5 -> 51.1 mm
- net SECOND_FIRE: track 40.9 -> 32.6 mm
- net THIRD_FIRE: track 28.8 -> 35.7 mm
- net GND: track 49.1 -> 55.3 mm
- net N$1: track 20.4 -> 15.7 mm
- net UP: track 25.9 -> 28.5 mm
- net CLK: track 20.2 -> 17.9 mm
- net LATCH: track 14.3 -> 16.1 mm
- net DATA: track 12.9 -> 14.4 mm
- net FIRE: track 32.4 -> 33.8 mm
- net DOWN: track 33.4 -> 33.3 mm, vias 0 -> 1
