File: hardware/atari2600-rtc/rtc.sch (EAGLE design)
At the start: 4 parts

Commit message: Update RTC design
Parts:
- added G1: CR2032H, battery:CR2032H
- added IC1: DS1307, ic-package:DIL8
Connections:
- new net N$4: G1.+, IC1.3
- net GND: now also G1.-, IC1.4
- net N$1: now also IC1.5
- net N$2: now also IC1.6
- net VCC: now also IC1.8
Other:
- moved on the sheet: R1, R2
Changed lines of the file:
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@@
 <part name="GND2" library="supply1" library_urn="urn:adsk.eagle:library:371" deviceset="GND" device=""/>
 <part name="GND3" library="supply1" library_urn="urn:adsk.eagle:library:371" deviceset="GND" device=""/>
-<part name="GND4" library="supply1" library_urn="urn:adsk.eagle:library:371" deviceset="GND" device=""/>
 <part name="P+1" library="supply1" library_urn="urn:adsk.eagle:library:371" deviceset="VCC" device=""/>
 <part name="P+2" library="supply1" library_urn="urn:adsk.eagle:library:371" deviceset="VCC" device=""/>
@@
 <part name="R1" library="rcl" library_urn="urn:adsk.eagle:library:334" deviceset="R-EU_" device="0204/7" package3d_urn="urn:adsk.eagle:package:23498/2" value="10k"/>
 <part name="R2" library="rcl" library_urn="urn:adsk.eagle:library:334" deviceset="R-EU_" device="0204/7" package3d_urn="urn:adsk.eagle:package:23498/2" value="10k"/>
+<part name="IC1" library="ic-package" library_urn="urn:adsk.eagle:library:239" deviceset="DIL8" device="" package3d_urn="urn:adsk.eagle:package:29519/2" value="DS1307"/>
+<part name="P+3" library="supply1" library_urn="urn:adsk.eagle:library:371" deviceset="VCC" device=""/>
+<part name="G1" library="battery" library_urn="urn:adsk.eagle:library:109" deviceset="CR2032H" device="" package3d_urn="urn:adsk.eagle:package:4585/1"/>
 </parts>
 <sheets>
@@
 <attribute name="VALUE" x="124.46" y="68.58" size="1.778" layer="96" rot="R90"/>
 </instance>
-<instance part="GND3" gate="1" x="86.36" y="73.66" smashed="yes">
-<attribute name="VALUE" x="83.82" y="71.12" size="1.778" layer="96"/>
+<instance part="GND3" gate="1" x="66.04" y="73.66" smashed="yes">
+<attribute name="VALUE" x="63.5" y="71.12" size="1.778" layer="96"/>
 </instance>
-<instance part="GND4" gate="1" x="55.88" y="88.9" smashed="yes" rot="R270">
-<attribute name="VALUE" x="53.34" y="91.44" size="1.778" layer="96" rot="R270"/>
+<instance part="P+1" gate="VCC" x="101.6" y="106.68" smashed="yes">
+<attribute name="VALUE" x="99.06" y="104.14" size="1.778" layer="96" rot="R90"/>
 </instance>
-<instance part="P+1" gate="VCC" x="60.96" y="114.3" smashed="yes">
-<attribute name="VALUE" x="58.42" y="111.76" size="1.778" layer="96" rot="R90"/>
-</instance>
-<instance part="P+2" gate="VCC" x="86.36" y="111.76" smashed="yes">
-<attribute name="VALUE" x="83.82" y="109.22" size="1.778" layer="96" rot="R90"/>
+<instance part="P+2" gate="VCC" x="93.98" y="106.68" smashed="yes">
+<attribute name="VALUE" x="91.44" y="104.14" size="1.778" layer="96" rot="R90"/>
 </instance>
 <instance part="P+4" gate="VCC" x="104.14" y="71.12" smashed="yes" rot="R90">
@@
 <attribute name="VALUE" x="116.459" y="72.644" size="1.778" layer="96" rot="R90"/>
 </instance>
-<instance part="R1" gate="G$1" x="60.96" y="104.14" smashed="yes" rot="R90">
-<attribute name="NAME" x="59.4614" y="100.33" size="1.778" layer="95" rot="R90"/>
-<attribute name="VALUE" x="64.262" y="100.33" size="1.778" layer="96" rot="R90"/>
+<instance part="R1" gate="G$1" x="101.6" y="96.52" smashed="yes" rot="R90">
+<attribute name="NAME" x="100.1014" y="92.71" size="1.778" layer="95" rot="R90"/>
+<attribute name="VALUE" x="104.902" y="92.71" size="1.778" layer="96" rot="R90"/>
 </instance>
-<instance part="R2" gate="G$1" x="99.06" y="96.52" smashed="yes" rot="R90">
-<attribute name="NAME" x="97.5614" y="92.71" size="1.778" layer="95" rot="R90"/>
-<attribute name="VALUE" x="102.362" y="92.71" size="1.778" layer="96" rot="R90"/>
+<instance part="R2" gate="G$1" x="93.98" y="96.52" smashed="yes" rot="R90">
+<attribute name="NAME" x="92.4814" y="92.71" size="1.778" layer="95" rot="R90"/>
+<attribute name="VALUE" x="97.282" y="92.71" size="1.778" layer="96" rot="R90"/>
+</instance>
+<instance part="IC1" gate="G$1" x="76.2" y="93.98" smashed="yes">
+<attribute name="NAME" x="71.755" y="98.425" size="1.778" layer="95"/>
+<attribute name="VALUE" x="71.755" y="85.09" size="1.778" layer="96"/>
+</instance>
+<instance part="P+3" gate="VCC" x="86.36" y="106.68" smashed="yes">
+<attribute name="VALUE" x="83.82" y="104.14" size="1.778" layer="96" rot="R90"/>
+</instance>
+<instance part="G1" gate="1" x="55.88" y="83.82" smashed="yes" rot="R90">
+<attribute name="NAME" x="52.705" y="81.28" size="1.778" layer="95" rot="R90"/>
+<attribute name="VALUE" x="60.96" y="81.28" size="1.778" layer="96" rot="R90"/>
 </instance>
 </instances>
@@
 </segment>
 <segment>
-<pinref part="P+2" gate="VCC" pin="VCC"/>
-<wire x1="86.36" y1="109.22" x2="86.36" y2="104.14" width="0.1524" layer="91"/>
-<wire x1="86.36" y1="104.14" x2="86.36" y2="101.6" width="0.1524" layer="91"/>
-<wire x1="86.36" y1="104.14" x2="99.06" y2="104.14" width="0.1524" layer="91"/>
-<junction x="86.36" y="104.14"/>
-<pinref part="R2" gate="G$1" pin="2"/>
-<wire x1="99.06" y1="104.14" x2="99.06" y2="101.6" width="0.1524" layer="91"/>
-</segment>
-<segment>
 <pinref part="P+1" gate="VCC" pin="VCC"/>
 <pinref part="R1" gate="G$1" pin="2"/>
-<wire x1="60.96" y1="111.76" x2="60.96" y2="109.22" width="0.1524" layer="91"/>
+<wire x1="101.6" y1="104.14" x2="101.6" y2="101.6" width="0.1524" layer="91"/>
 </segment>
 <segment>
@@
 <pinref part="C1" gate="G$1" pin="1"/>
 <wire x1="106.68" y1="71.12" x2="109.22" y2="71.12" width="0.1524" layer="91"/>
+</segment>
+<segment>
+<pinref part="R2" gate="G$1" pin="2"/>
+<pinref part="P+2" gate="VCC" pin="VCC"/>
+<wire x1="93.98" y1="101.6" x2="93.98" y2="104.14" width="0.1524" layer="91"/>
+</segment>
+<segment>
+<pinref part="P+3" gate="VCC" pin="VCC"/>
+<wire x1="86.36" y1="104.14" x2="86.36" y2="96.52" width="0.1524" layer="91"/>
+<pinref part="IC1" gate="G$1" pin="8"/>
+<wire x1="86.36" y1="96.52" x2="83.82" y2="96.52" width="0.1524" layer="91"/>
 </segment>
 </net>
@@
 </segment>
 <segment>
-<pinref part="GND4" gate="1" pin="GND"/>
-<wire x1="58.42" y1="88.9" x2="63.5" y2="88.9" width="0.1524" layer="91"/>
-<wire x1="63.5" y1="88.9" x2="66.04" y2="88.9" width="0.1524" layer="91"/>
-<wire x1="63.5" y1="88.9" x2="63.5" y2="93.98" width="0.1524" layer="91"/>
-<junction x="63.5" y="88.9"/>
-<wire x1="63.5" y1="93.98" x2="66.04" y2="93.98" width="0.1524" layer="91"/>
-<wire x1="63.5" y1="88.9" x2="63.5" y2="86.36" width="0.1524" layer="91"/>
-<wire x1="63.5" y1="86.36" x2="66.04" y2="86.36" width="0.1524" layer="91"/>
-<wire x1="63.5" y1="86.36" x2="63.5" y2="83.82" width="0.1524" layer="91"/>
-<junction x="63.5" y="86.36"/>
-<wire x1="63.5" y1="83.82" x2="66.04" y2="83.82" width="0.1524" layer="91"/>
+<pinref part="GND2" gate="1" pin="GND"/>
+<pinref part="C1" gate="G$1" pin="2"/>
+<wire x1="119.38" y1="71.12" x2="116.84" y2="71.12" width="0.1524" layer="91"/>
 </segment>
 <segment>
 <pinref part="GND3" gate="1" pin="GND"/>
-<wire x1="86.36" y1="76.2" x2="86.36" y2="78.74" width="0.1524" layer="91"/>
-</segment>
-<segment>
-<pinref part="GND2" gate="1" pin="GND"/>
-<pinref part="C1" gate="G$1" pin="2"/>
-<wire x1="119.38" y1="71.12" x2="116.84" y2="71.12" width="0.1524" layer="91"/>
+<wire x1="66.04" y1="76.2" x2="66.04" y2="88.9" width="0.1524" layer="91"/>
+<pinref part="IC1" gate="G$1" pin="4"/>
+<wire x1="66.04" y1="88.9" x2="68.58" y2="88.9" width="0.1524" layer="91"/>
+<pinref part="G1" gate="1" pin="-"/>
+<wire x1="55.88" y1="78.74" x2="55.88" y2="76.2" width="0.1524" layer="91"/>
+<wire x1="55.88" y1="76.2" x2="66.04" y2="76.2" width="0.1524" layer="91"/>
+<junction x="66.04" y="76.2"/>
 </segment>
 </net>
@@
 <segment>
 <pinref part="X1" gate="G$1" pin="3"/>
-<wire x1="106.68" y1="88.9" x2="99.06" y2="88.9" width="0.1524" layer="91"/>
+<wire x1="106.68" y1="88.9" x2="93.98" y2="88.9" width="0.1524" layer="91"/>
 <pinref part="R2" gate="G$1" pin="1"/>
-<wire x1="99.06" y1="88.9" x2="93.98" y2="88.9" width="0.1524" layer="91"/>
-<wire x1="99.06" y1="88.9" x2="99.06" y2="91.44" width="0.1524" layer="91"/>
-<junction x="99.06" y="88.9"/>
+<wire x1="93.98" y1="88.9" x2="93.98" y2="91.44" width="0.1524" layer="91"/>
+<junction x="93.98" y="88.9"/>
+<pinref part="IC1" gate="G$1" pin="5"/>
+<wire x1="83.82" y1="88.9" x2="93.98" y2="88.9" width="0.1524" layer="91"/>
 </segment>
 </net>
@@
 <segment>
 <pinref part="X1" gate="G$1" pin="4"/>
-<wire x1="106.68" y1="86.36" x2="93.98" y2="86.36" width="0.1524" layer="91"/>
-<wire x1="93.98" y1="86.36" x2="93.98" y2="68.58" width="0.1524" layer="91"/>
-<wire x1="93.98" y1="68.58" x2="50.8" y2="68.58" width="0.1524" layer="91"/>
-<wire x1="50.8" y1="68.58" x2="50.8" y2="96.52" width="0.1524" layer="91"/>
-<wire x1="50.8" y1="96.52" x2="60.96" y2="96.52" width="0.1524" layer="91"/>
+<wire x1="106.68" y1="86.36" x2="101.6" y2="86.36" width="0.1524" layer="91"/>
 <pinref part="R1" gate="G$1" pin="1"/>
-<wire x1="60.96" y1="96.52" x2="66.04" y2="96.52" width="0.1524" layer="91"/>
-<wire x1="60.96" y1="99.06" x2="60.96" y2="96.52" width="0.1524" layer="91"/>
-<junction x="60.96" y="96.52"/>
+<wire x1="101.6" y1="86.36" x2="101.6" y2="91.44" width="0.1524" layer="91"/>
+<wire x1="101.6" y1="86.36" x2="86.36" y2="86.36" width="0.1524" layer="91"/>
+<junction x="101.6" y="86.36"/>
+<wire x1="86.36" y1="86.36" x2="86.36" y2="91.44" width="0.1524" layer="91"/>
+<pinref part="IC1" gate="G$1" pin="6"/>
+<wire x1="86.36" y1="91.44" x2="83.82" y2="91.44" width="0.1524" layer="91"/>
 </segment>
 </net>
+<net name="N$4" class="0">
+<segment>
+<pinref part="G1" gate="1" pin="+"/>
+<wire x1="55.88" y1="88.9" x2="55.88" y2="91.44" width="0.1524" layer="91"/>
+<pinref part="IC1" gate="G$1" pin="3"/>
+<wire x1="55.88" y1="91.44" x2="68.58" y2="91.44" width="0.1524" layer="91"/>
+</segment>
+</net>

Commit message: Update RTC design
Parts:
- removed G1: CR2032H, battery:CR2032H
- added Q1: (no value), crystal:CRYSTALTC26V
- added U$1: CR2032, cr2032:CR2032
Connections:
- new net N$3: IC1.3, U$1.VCC
- new net N$5: IC1.1, Q1.2
- net GND: now also U$1.GND; no longer G1.-
- net N$4: now also IC1.2, Q1.1; no longer G1.+, IC1.3
Other:
- moved on the sheet: C1, IC1, R1, R2, X1

Commit message: Change battery socket in RTC design
Parts:
- removed U$1: CR2032, cr2032:CR2032
- added BT1: (no value), SparkFun-Batteries:BATTERY-20MM_PTH
Connections:
- net GND: now also BT1.-; no longer U$1.GND
- net N$3: now also BT1.+; no longer U$1.VCC
